Commit message: removed reference to meshes to avoid errors with locating the mesh files. these were not necessary anyways

File: robosuite/controllers/dynamics/dynamic_models/iiwa14/iiwa14.urdf (robot description, URDF)
Before this commit: robot iiwa14, 11 links, 10 joints
Links:
- link lbr_link_0: geometry 
- link lbr_link_1: geometry 
- link lbr_link_2: geometry 
- link lbr_link_3: geometry 
- link lbr_link_4: geometry 
- link lbr_link_5: geometry 
- link lbr_link_6: geometry 
- link lbr_link_7: geometry 
- link lbr_link_ee: geometry 

Commit message: updated the parameters of the nominal iiwa14dynamics  model

File: robosuite/controllers/dynamics/dynamic_models/iiwa14/iiwa14.urdf (robot description, URDF)
Before this commit: robot iiwa14, 11 links, 10 joints
Links:
- added link lbr_link_ee2, mass 0.14730
- link lbr_link_ee: mass 0.39127 -> 0.245
Joints:
- added joint lbr_joint_ee_mid: type fixed, parent lbr_link_ee, child lbr_link_ee2, origin xyz=0 0 0.0375 rpy=0 0 0
- joint lbr_joint_tcp: parent lbr_link_ee -> lbr_link_ee2

Commit message: Revert "updated the parameters of the nominal iiwa14dynamics  model"
This reverts commit 63ab69cb3eb2e118520cfe53ba1b2200b10530c4.

File: robosuite/controllers/dynamics/dynamic_models/iiwa14/iiwa14.urdf (robot description, URDF)
Before this commit: robot iiwa14, 12 links, 11 joints
Links:
- removed link lbr_link_ee2
- link lbr_link_ee: mass 0.245 -> 0.39127
Joints:
- removed joint lbr_joint_ee_mid
- joint lbr_joint_tcp: parent lbr_link_ee2 -> lbr_link_ee

Commit message: rotated joint_ee in the iiwa14 urdf to reflect the mujoco model

File: robosuite/controllers/dynamics/dynamic_models/iiwa14/iiwa14.urdf (robot description, URDF)
Before this commit: robot iiwa14, 12 links, 11 joints
Joints:
- joint lbr_joint_ee: origin xyz=0 0 0.045 rpy=0 0 0 -> xyz=0 0 0.045 rpy=0 0 3.141592653589793

Commit message: corrected joint origin xyz for lbr_joint_tcp

File: robosuite/controllers/dynamics/dynamic_models/iiwa14/iiwa14.urdf (robot description, URDF)
Before this commit: robot iiwa14, 12 links, 11 joints
Joints:
- joint lbr_joint_tcp: origin xyz=0 0 0.0995 rpy=0 0 0 -> xyz=0 0 0.062 rpy=0 0 0
